File: NMEA2000-COMMON.kicad_pcb (KiCad board)
At the start: 2 copper layers, 100 x 85 mm, 62 parts, among them J2 CAN, SW1 PRG, SW2 INSTANCE, SW3 BUS, U1 MCP2551-I-P, U2 TMR-2-2411, U3 74HCT595, U4 74HCT595, U5 Teensy_4.0

Commit message: Revise INSTANCE
Connections:
- net /CH0 renamed /D23
- net /CH1 renamed /D22
- net /CH2 renamed /D21
- net /CH3 renamed /D20
- net /CH4 renamed /D19
- net /CH5 renamed /D18
- net /CH6 renamed /D17
- net /CH7 renamed /D16

Commit message: PISI update
Parts:
- added C101: 100nF, Capacitor_SMD:C_0805_2012Metric, F.Cu at (95.2, 42.9)
- added R101: 4K7 0.125W, Resistor_SMD:R_0805_2012Metric, F.Cu at (111.3, 25.5)
- added R102: 4K7 0.125W, Resistor_SMD:R_0805_2012Metric, F.Cu at (108.8, 25.5)
- added R103: 4K7 0.125W, Resistor_SMD:R_0805_2012Metric, F.Cu at (106.2, 25.5)
- added R104: 4K7 0.125W, Resistor_SMD:R_0805_2012Metric, F.Cu at (103.7, 25.5)
- added R105: 4K7 0.125W, Resistor_SMD:R_0805_2012Metric, F.Cu at (101.1, 25.5)
- added R106: 4K7 0.125W, Resistor_SMD:R_0805_2012Metric, F.Cu at (98.6, 25.5)
- added R107: 4K7 0.125W, Resistor_SMD:R_0805_2012Metric, F.Cu at (96.1, 25.5)
- added R108: 4K7 0.125W, Resistor_SMD:R_0805_2012Metric, F.Cu at (93.5, 25.5)
- added U101: 74LS165, Package_SO:SO-16_3.9x9.9mm_P1.27mm, F.Cu at (100.1, 37.5)
- moved C4 9.41 mm to (95.2, 54.9)
- moved U4 9.41 mm to (100.1, 49.5)
- moved U3 9.10 mm to (100.1, 61.5)
- moved C2 9.09 mm to (95.2, 66.9)
- moved SW1 0.57 mm to (61.2, 24.4)
Connections:
- net /MPX_LATCH renamed /LED_LATCH
- net /MPX_SER renamed /LED_SER
- SW2 pad 1: /ADDR_0 -> Net-(R108-Pad2)
- SW2 pad 2: /ADDR_1 -> Net-(R107-Pad2)
- SW2 pad 3: /ADDR_2 -> Net-(R106-Pad2)
- SW2 pad 4: /ADDR_3 -> Net-(R105-Pad2)
- SW2 pad 5: /ADDR_4 -> Net-(R104-Pad2)
- SW2 pad 6: /ADDR_5 -> Net-(R103-Pad2)
- SW2 pad 7: /ADDR_6 -> Net-(R102-Pad2)
- SW2 pad 8: /ADDR_7 -> Net-(R101-Pad2)
- U3 pad 11: /MPX_CLOCK -> /LED_CLOCK
- U4 pad 11: /MPX_CLOCK -> /LED_CLOCK
- U4 pad 14: /MPX_DATA -> /LED_DATA
- U5 pad 10: /ADDR_4 -> /D8
- U5 pad 11: /ADDR_3 -> /INSTANCE_CE
- U5 pad 12: /ADDR_2 -> /INSTANCE_Q7
- U5 pad 13: /ADDR_1 -> /INSTANCE_PL
- U5 pad 14: /ADDR_0 -> /INSTANCE_CP
- U5 pad 2: /MPX_CLOCK -> /LED_DATA
- U5 pad 4: /MPX_DATA -> /LED_CLOCK
- U5 pad 7: /ADDR_7 -> /D5
- U5 pad 8: /ADDR_6 -> /D6
- U5 pad 9: /ADDR_5 -> /D7
Routing:
- net +5V: track 219.5 -> 262.8 mm
- net /ADDR_7: track 33.3 -> 0.00 mm
- net /D8: track 0.00 -> 30.9 mm
- net /MPX_CLOCK: track 29.1 -> 0.00 mm, vias 2 -> 0
- net /ADDR_6: track 28.9 -> 0.00 mm
- net /INSTANCE_CP: track 0.00 -> 28.8 mm, vias 0 -> 1
- net /D7: track 0.00 -> 27.6 mm
- net /INSTANCE_PL: track 0.00 -> 27.0 mm, vias 0 -> 1
- net /LED_CLOCK: track 0.00 -> 24.6 mm, vias 0 -> 2
- net /ADDR_5: track 24.4 -> 0.00 mm
- net /D6: track 0.00 -> 24.2 mm
- net /D5: track 0.00 -> 20.9 mm
- net /ADDR_4: track 19.9 -> 0.00 mm
- net /MPX_DATA: track 17.6 -> 0.00 mm, vias 1 -> 0
- net Net-(R101-Pad2): track 0.00 -> 17.3 mm
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
Commit message: Tidy up
Connections:
- J2 pad 4: /CAN_L -> Net-(J2-Pad4)
- J2 pad 5: /CAN_SCR -> Net-(J2-Pad5)
- R2 pad 2: /CAN_H -> Net-(R2-Pad2)
- SW3 pad 1: /CAN_H -> Net-(J2-Pad5)
- SW3 pad 2: GND -> Net-(R2-Pad2)
- SW3 pad 3: /CAN_SCR -> Net-(J2-Pad4)
- SW3 pad 4: /CAN_L -> GND
- U1 pad 6: /CAN_L -> Net-(J2-Pad4)
Routing:
- net Net-(J2-Pad4): track 0.00 -> 50.3 mm
- net /CAN_L: track 46.9 -> 0.00 mm
- net /CAN_SCR: track 35.2 -> 0.00 mm
- net Net-(J2-Pad5): track 0.00 -> 30.8 mm
- net Net-(R2-Pad2): track 0.00 -> 12.5 mm
- net /CAN_H: track 4.22 -> 0.00 mm

Commit message: Tidy up.
Parts:
- R101, R102, R103, R104, R105, R106, R107, R108: moved to B.Cu
- moved R101 0.13 mm to (111.3, 25.7)
- moved R102 0.13 mm to (108.8, 25.7)
- moved R103 0.13 mm to (106.2, 25.7)
- moved R104 0.13 mm to (103.7, 25.7)
- moved R105 0.13 mm to (101.1, 25.7)
- moved R106 0.13 mm to (98.6, 25.7)
- moved R107 0.13 mm to (96.1, 25.7)
- moved R108 0.13 mm to (93.5, 25.7)
Routing:
- net /D5: track 20.9 -> 18.1 mm, vias 0 -> 1
- net /D6: track 24.2 -> 21.7 mm, vias 0 -> 1
- net /D7: track 27.6 -> 25.3 mm, vias 0 -> 1
- net /D8: track 30.9 -> 28.9 mm, vias 0 -> 1
- net /D16: track 33.8 -> 35.5 mm, vias 0 -> 1
- net /D17: track 30.5 -> 32.0 mm, vias 0 -> 1
- net /D18: track 27.2 -> 28.4 mm, vias 0 -> 1
- net +5V: track 262.8 -> 264.0 mm, vias 1 -> 2
- net /D19: track 23.9 -> 24.9 mm, vias 0 -> 1
- net /D20: track 21.7 -> 22.4 mm, vias 0 -> 1
- net /D23: track 11.0 -> 10.5 mm, vias 0 -> 1
- net /D21: track 17.6 -> 17.8 mm, vias 0 -> 1
- net /D22: track 14.0 -> 14.1 mm, vias 0 -> 1
- net /TRANSMIT_LED: vias 0 -> 1
