File: hardware/NMEA2000-COMMON.sch (KiCad schematic (older format))
At the start: 67 parts, among them J2 CAN, Q1 BSS138, Q2 BSS138, SW1 PRG, SW2 INSTANCE, SW3 BUS, U1 MCP2551-I-P, U101 74HC165, U2 TMR-2-2411, U3 74HCT595, U4 74HCT595, U5 Teensy_4.0

Commit message: Stuff
Parts:
- U101: symbol pdjr:74LS165 -> NMEA2000-COMMON-rescue:74LS165-pdjr
- U2: symbol pdjr:TMR-2-2411 -> NMEA2000-COMMON-rescue:TMR-2-2411-pdjr
- U5: symbol pdjr:Teensy_3.2 -> NMEA2000-COMMON-rescue:Teensy_3.2-pdjr
Connections:
- wire segments 281 -> 275
Changed lines of the file:
@@
 	1    0    0    -1
 $EndComp
-Connection ~ 8450 3450
 Text Label 10150 2500 2    50   ~ 0
 PRG
@@
 Wire Wire Line
 	10300 5950 10400 5950
-Connection ~ 8450 4950
 $Comp
 L Device:CP_Small C2
@@
 NoConn ~ 3600 4550
 $Comp
-L pdjr:Teensy_3.2 U5
+L NMEA2000-COMMON-rescue:Teensy_3.2-pdjr U5
 U 1 1 60F2AB82
 P 4150 6050
@@
 CAN_SCR
 $Comp
-L pdjr:TMR-2-2411 U2
+L NMEA2000-COMMON-rescue:TMR-2-2411-pdjr U2
 U 1 1 63A71732
 P 3500 1150
@@
 	8450 850  8450 950
 $Comp
-L pdjr:74LS165 U101
+L NMEA2000-COMMON-rescue:74LS165-pdjr U101
 U 1 1 63F7C7A4
 P 8450 1850
@@
 	7550 5700 8050 5700
 Wire Wire Line
-	8450 3450 11000 3450
-Wire Wire Line
 	7850 5000 7850 4950
-Connection ~ 7850 4950
 Wire Wire Line
 	7850 5200 7850 6250
@@
 	8850 5950 10000 5950
 Wire Wire Line
-	8450 4950 11000 4950
-Wire Wire Line
 	8450 4750 11000 4750
 Wire Wire Line
-	11000 3450 11000 3750
-Connection ~ 11000 3750
-Wire Wire Line
 	11000 3750 11000 3850
-Wire Wire Line
-	8350 4950 8450 4950
-Wire Wire Line
-	7850 4950 8450 4950
 Connection ~ 11000 3850
 Wire Wire Line
@@
 Wire Wire Line
 	11000 4450 11000 4750
-Connection ~ 11000 4750
-Wire Wire Line
-	11000 4750 11000 4950
-Connection ~ 11000 4950
-Wire Wire Line
-	11000 4950 11000 5250
-Connection ~ 11000 5250
 Wire Wire Line
 	11000 5250 11000 5350
@@
 	3000 950  2650 950
 Connection ~ 2650 950
+Wire Wire Line
+	7850 4950 8450 4950
+Connection ~ 7850 4950
 $EndSCHEMATC

Commit message: Tweak
Connections:
- net labels added: PISO_CP, PISO_PL, PISO_Q7, SIPO_CLOCK, SIPO_DATA, SIPO_LATCH
- net labels removed: INSTANCE_CP, INSTANCE_PL, INSTANCE_Q7, LED_CLOCK, LED_DATA, LED_LATCH
Changed lines of the file:
@@
 	10300 4250 10400 4250
 Text Label 7550 3750 2    50   ~ 0
-LED_DATA
+SIPO_DATA
 Text Label 7550 4000 2    50   ~ 0
-LED_CLOCK
+SIPO_CLOCK
 Text Label 7550 4200 2    50   ~ 0
-LED_LATCH
+SIPO_LATCH
 Wire Wire Line
 	8450 4650 8450 4750
@@
 	10300 5750 10400 5750
 Text Label 7550 5500 2    50   ~ 0
-LED_CLOCK
+SIPO_CLOCK
 Text Label 7550 5700 2    50   ~ 0
-LED_LATCH
+SIPO_LATCH
 Wire Wire Line
 	8450 6150 8450 6250
@@
 PRG
 Text Label 4150 5750 0    50   ~ 0
-LED_CLOCK
+SIPO_CLOCK
 Text Label 4150 5950 0    50   ~ 0
-LED_DATA
+SIPO_DATA
 Text Label 4150 5850 0    50   ~ 0
-LED_LATCH
+SIPO_LATCH
 Text Label 3050 5150 2    50   ~ 0
 D17
@@
 $EndComp
 Text Label 7550 1750 2    50   ~ 0
-INSTANCE_CP
+PISO_CP
 Text Label 7550 1250 2    50   ~ 0
-INSTANCE_Q7
+PISO_Q7
 Text Label 7550 1550 2    50   ~ 0
-INSTANCE_PL
+PISO_PL
 Text Label 4150 4850 0    50   ~ 0
-INSTANCE_PL
+PISO_PL
 Text Label 4150 4750 0    50   ~ 0
-INSTANCE_CP
+PISO_CP
 Text Label 4150 4950 0    50   ~ 0
-INSTANCE_Q7
+PISO_Q7
 Text Label 4150 5050 0    50   ~ 0
 D9

Commit message: Relay
Parts:
- U3, U4: symbol 74xx:74HC595 -> NMEA2000-COMMON-rescue:74HC595-74xx
Changed lines of the file:
@@
 $EndComp
 $Comp
-L 74xx:74HC595 U4
+L NMEA2000-COMMON-rescue:74HC595-74xx U4
 U 1 1 6338D277
 P 8450 4150
@@
 $EndComp
 $Comp
-L 74xx:74HC595 U3
+L NMEA2000-COMMON-rescue:74HC595-74xx U3
 U 1 1 6399F1E7
 P 8450 5650
