File: hardware/NMEA2000-COMMON.sch (KiCad schematic (older format))
At the start: 67 parts, among them J2 CAN, Q1 BSS138, Q2 BSS138, SW1 PRG, SW2 INSTANCE, SW3 BUS, U1 MCP2551-I-P, U101 74HC165, U2 TMR-2-2411, U3 74HCT595, U4 74HCT595, U5 Teensy_4.0

Commit message: Fix
Connections:
- wire segments 275 -> 288
