File: hardware/NMEA2000-COMMON.kicad_pcb (KiCad board)
At the start: 2 copper layers, 100 x 85 mm, 74 parts, among them J2 CAN, Q1 BSS138, Q2 BSS138, SW1 PRG, SW2 INSTANCE, SW3 BUS, U1 MCP2551-I-P, U101 74HC165, U2 TMR-2-2411, U3 74HCT595, U4 74HCT595, U5 Teensy_4.0

Commit message: Fix
Connections:
- net /D16 renamed D16
- net /D17 renamed D17
- net /D18 renamed D18
- net /D19 renamed D19
- net /D20 renamed D20
- net /D21 renamed D21
- net /D22 renamed D22
- net /D23 renamed D23
- net /D5 renamed D5
- net /D6 renamed D6
- net /D7 renamed D7
- net /D8 renamed D8
- net /D9 renamed D9
